File: hardware/PCB_EU_LITE/PCB_EU_LITE.kicad_pcb (KiCad board)
At the start: 4 copper layers, 100 x 100 mm, 167 parts, among them J101 24 V IN, J201 UART 3V3, J301 MEM2061 SPI, J401 SHT4x XH2.54-4P-90, J403 FLOAT / GND, J411 FAN1 2510-4P 90deg, J421 FAN2 2510-4P 90deg, J501 LED + / GND, J502 LED 2 + / GND, J503 LED 3 + / GND, J701 PTC + / RETURN, J702 PUMP + / RETURN, Q102 IRL2505, Q411 FAN1 AO3422, Q421 FAN2 AO3422, Q501 BSC146N10LS5, Q701 BC847B-DIO, Q702 BC857B, Q703 CSD19531KCS, Q704 AO3422, Q901 BC847B (R), Q902 BC847B (G), Q903 BC847B (B), SW201 RESET, SW202 BOOT, U101 ST1S14PHR, U102 INA238, U201 ST1S10PHR, U202 ESP32-WROOM-32E-N4, U301 MCP7940N, U401 USBLC6-2SC6, U501 LM3429MH/NOPB, Y301 32.768k CL7p

Commit message: Release verified r3 Gerber package and align F103 value
Parts:
- F103: value 6.3 A slow -> 6.3 A fast
Changed lines of the file:
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@@
 			)
 		)
-		(property "Value" "6.3 A slow"
+		(property "Value" "6.3 A fast"
 			(at 0 5 0)
 			(layer "F.Fab")
