File: hardware/PCB_EU_LITE/LED.kicad_sch (KiCad schematic)
At the start: 40 parts, among them J501 LED + / GND, J502 LED 2 + / GND, J503 LED 3 + / GND, Q501 BSC146N10LS5, U501 LM3429MH/NOPB

Commit message: Apply the 283 kHz LED transition to sources, model and docs
Set R507 to 82k and R506 to 1k in the generator, regenerate the schematic,
design.json and BOM, and carry the new operating point (283.45 kHz,
1.444 A, 69.3 W) through verify.py, the power-stage model and the docs.
Only the Value fields of R506/R507 change on the board; geometry, nets and
silkscreen are untouched.

The procurement blocker is resolved: 82k is already in the 2026-10-23
catalogue snapshot and is now bought twice (R101 + R507); the 1k 1206 line
is added from the Salvats product page read on 2026-10-27 and preserved on
refresh through snapshot_prices.SITE_QUOTES. Purchase total is unchanged at
38.49 EUR with no unpriced lines.

verify.py (58 checks), its mutation tests, the boost-model tests, the price
refresh test, check_schematics.py and check_standalone.py pass. KiCad DRC,
board parity, fabricate.py and a new Gerber set were NOT run: no pcbnew,
Shapely or gerbonara in this environment. Gerber r3 stays historical and the
bench programme is still open.

Co-Authored-By: Claude Opus 5 <noreply@anthropic.com>
Claude-Session: https://claude.ai/code/session_01YbDYdPzNZ5NsoW89vkngV3
Parts:
- R505: Design_note With R506=620R: 5.32k total, ~1.55 A / 75 W-class at 48 V s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 -> With R506=1k: 5.7k total, ~1.444 A / 69.3 W-class at 48 V s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
- R506: value 620R 1% -> 1k 1%; MPN CRCW1206620RFKTABC -> SMD1206-1K-1%
- R507: value 56k 1% -> 82k 1%; MPN SMD1206 56K 1% -> CRCW120682K0FKTABC
Other:
- note added: "J501/J502/J503 are parallel outputs AFTER R502: one 69 W-class LED channel, ~1.444 A TOTAL at ~48 V (1.235 V x 1k / (5.7k x 0.15 R)). LM3429 VIN senses the actual 24 V input. RCT is fed from SW through 82k + 6k2, CT 1 nF C0G: 25 / (88.2k x 1 nF) = 283.45 kHz nominal (EU-0.1 LED1 used 56k = 402 kHz). L501: stock Feryster DTMSS-27/0.047/15-V, 47 uH, 15 A, standing toroid ~35 mm high. Model peak <=4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"
- note removed: "J501/J502/J503 are parallel outputs AFTER R502: one 75 W-class LED channel, ~1.55 A TOTAL at ~48 V (1.235 V x 1k / (5.32k x 0.15 R)). LM3429 VIN senses the actual 24 V input. RCT is fed from SW through 56k + 6k2, CT 1 nF C0G: same as EU-0.1 LED1 (frequency unchanged). L501: stock Feryster DTMSS-27/0.047/15-V, 47 uH, 15 A, standing toroid ~35 mm high. Model peak <=4.36 A at 21.6 V, 90% efficiency,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"
Changed lines of the file:
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@@
 (kicad_sch (version 20260306) (generator "eeschema") (generator_version "10.0") (paper "A3") (title_block (title "06 | LED boost channel (LM3429, one channel)") (date "2026-10-24") (rev "EU-LITE-0.1") (company "GrowBox | EU-LITE from stock") (comment 1 "SCHEMATIC DRAFT | no PCB / manufacturing release"))
 (text "06 | LED boost channel (LM3429, one channel)" (at 12.7 12.7 0) (effects (font (size 2 2)) (justify left top)))
-(text "J501/J502/J503 are parallel outputs AFTER R502: one 75 W-class LED channel, ~1.55 A TOTAL at ~48 V (1.235 V x 1k / (5.32k x 0.15 R)).\nLM3429 VIN senses the actual 24 V input. RCT is fed from SW through 56k + 6k2, CT 1 nF C0G: same as EU-0.1 LED1 (frequency unchanged).\nL501: stock Feryster DTMSS-27/0.047/15-V, 47 uH, 15 A, standing toroid ~35 mm high. Model peak <=4.36 A at 21.6 V, 90% efficiency, 43.5 uH, 1.26 V CSH and 1% resistors.\nLM3429 IS threshold is 215/245/275 mV min/typ/max (TI Rev H): minimum limit 5.32 A with R501=40 mOhm +1%; modeled current-limit headroom >=20%. Verify real tolerances and heating.\nQ501: stock BSC146N10LS5 (TDSON-8, 100 V, 14.6 mOhm, Qgd 2.8 nC) on the LM3429 7 V gate drive; no heatsink. The 75 W setpoint needs wide power copper, thermal vias and temperature checks.\nGate resistor 2 x 10 R in parallel = 5 R (stock) instead of 4.7 R. D501: stock SBRT15U100SP5 (100 V, 15 A, PowerDI5): pad 1 cathode, pads 2 anode.\nHSP/HSN use equal 1k filters; output bank is BEFORE the LED shunt; LED negative is GND. OVP = 1.24 V x 44 = 54.56 V; 63 V electrolytic and 100 V ceramics.\nnDIM: GPIO25 -> 5.1k -> nDIM, 10k to GND (HIGH 2.19 V, Hi-Z 0.6 V). No BAT54/LM2903 hardware block (see 02 | UVLO note).\nRequired firmware setting: at 1 kHz / 8 bit use >=5 PWM counts (19.53 us); the new startup-pulse estimate is ~16 us at 21.6 V / 48 V. Firmware is not changed here.\nBoost output has a DC path from VIN even while disabled. Fuse is not semiconductor short-circuit proof. 22u COMP intentionally slow." (at 12.7 251 0) (effects (font (size 1.02 1.02)) (justify left top)))
+(text "J501/J502/J503 are parallel outputs AFTER R502: one 69 W-class LED channel, ~1.444 A TOTAL at ~48 V (1.235 V x 1k / (5.7k x 0.15 R)).\nLM3429 VIN senses the actual 24 V input. RCT is fed from SW through 82k + 6k2, CT 1 nF C0G: 25 / (88.2k x 1 nF) = 283.45 kHz nominal (EU-0.1 LED1 used 56k = 402 kHz).\nL501: stock Feryster DTMSS-27/0.047/15-V, 47 uH, 15 A, standing toroid ~35 mm high. Model peak <=4.24 A at 21.6 V, 90% efficiency, 43.5 uH, 283.45 kHz, 1.26 V CSH and 1% resistors.\nLM3429 IS threshold is 215/245/275 mV min/typ/max (TI Rev H): minimum limit 5.32 A with R501=40 mOhm +1%; modeled current-limit headroom >=20%. Verify real tolerances and heating.\nQ501: stock BSC146N10LS5 (TDSON-8, 100 V, 14.6 mOhm, Qgd 2.8 nC) on the LM3429 7 V gate drive; no heatsink. The 69 W setpoint needs wide power copper, thermal vias and temperature checks.\nGate resistor 2 x 10 R in parallel = 5 R (stock) instead of 4.7 R. D501: stock SBRT15U100SP5 (100 V, 15 A, PowerDI5): pad 1 cathode, pads 2 anode.\nHSP/HSN use equal 1k filters; output bank is BEFORE the LED shunt; LED negative is GND. OVP = 1.24 V x 44 = 54.56 V; 63 V electrolytic and 100 V ceramics.\nnDIM: GPIO25 -> 5.1k -> nDIM, 10k to GND (HIGH 2.19 V, Hi-Z 0.6 V). No BAT54/LM2903 hardware block (see 02 | UVLO note).\nRequired firmware setting: at 1 kHz / 8 bit use >=5 PWM counts (19.53 us); the startup-pulse estimate at the 69 W setpoint is ~14.7 us at 21.6 V / 48 V. Firmware is not changed here.\nBoost output has a DC path from VIN even while disabled. Fuse is not semiconductor short-circuit proof. 22u COMP intentionally slow." (at 12.7 251 0) (effects (font (size 1.02 1.02)) (justify left top)))
 (symbol (lib_id "EU_LITE:LM3429") (at 85.09 59.69 0) (unit 1) (in_bom yes) (on_board yes) (dnp no)
 (property "Reference" "U501" (at 85.09 45.16 0) (effects (font (size 1.15 1.15)) ))
@@
 (property "MPN" "SMD1206 4K7 1%" (at 374.65 119.38 0) (effects (font (size 1 1)) (hide yes)))
 (property "Source" "buy" (at 374.65 119.38 0) (effects (font (size 1 1)) (hide yes)))
-(property "Design_note" "With R506=620R: 5.32k total, ~1.55 A / 75 W-class at 48 V shared by all LED outputs" (at 374.65 119.38 0) (effects (font (size 1 1)) (hide yes)))
+(property "Design_note" "With R506=1k: 5.7k total, ~1.444 A / 69.3 W-class at 48 V shared by all LED outputs" (at 374.65 119.38 0) (effects (font (size 1 1)) (hide yes)))
 (property "FootprintStatus" "PACKAGE ONLY - verify before PCB" (at 374.65 119.38 0) (effects (font (size 1 1)) (hide yes)))
 (pin "1")
@@
 (symbol (lib_id "EU_LITE:R") (at 45.72 139.7 0) (unit 1) (in_bom yes) (on_board yes) (dnp no)
 (property "Reference" "R506" (at 45.72 134.06 0) (effects (font (size 1.15 1.15)) ))
-(property "Value" "620R 1%" (at 45.72 145.34 0) (effects (font (size 0.98 0.98)) ))
+(property "Value" "1k 1%" (at 45.72 145.34 0) (effects (font (size 0.98 0.98)) ))
 (property "Footprint" "Resistor_SMD:R_1206_3216Metric" (at 45.72 139.7 0) (effects (font (size 1 1)) (hide yes)))
 (property "Datasheet" "" (at 45.72 139.7 0) (effects (font (size 1 1)) (hide yes)))
-(property "MPN" "CRCW1206620RFKTABC" (at 45.72 139.7 0) (effects (font (size 1 1)) (hide yes)))
+(property "MPN" "SMD1206-1K-1%" (at 45.72 139.7 0) (effects (font (size 1 1)) (hide yes)))
 (property "Source" "buy" (at 45.72 139.7 0) (effects (font (size 1 1)) (hide yes)))
 (property "Design_note" "" (at 45.72 139.7 0) (effects (font (size 1 1)) (hide yes)))
@@
 (symbol (lib_id "EU_LITE:R") (at 106.68 139.7 0) (unit 1) (in_bom yes) (on_board yes) (dnp no)
 (property "Reference" "R507" (at 106.68 134.06 0) (effects (font (size 1.15 1.15)) ))
-(property "Value" "56k 1%" (at 106.68 145.34 0) (effects (font (size 0.98 0.98)) ))
+(property "Value" "82k 1%" (at 106.68 145.34 0) (effects (font (size 0.98 0.98)) ))
 (property "Footprint" "Resistor_SMD:R_1206_3216Metric" (at 106.68 139.7 0) (effects (font (size 1 1)) (hide yes)))
 (property "Datasheet" "" (at 106.68 139.7 0) (effects (font (size 1 1)) (hide yes)))
-(property "MPN" "SMD1206 56K 1%" (at 106.68 139.7 0) (effects (font (size 1 1)) (hide yes)))
+(property "MPN" "CRCW120682K0FKTABC" (at 106.68 139.7 0) (effects (font (size 1 1)) (hide yes)))
 (property "Source" "buy" (at 106.68 139.7 0) (effects (font (size 1 1)) (hide yes)))
 (property "Design_note" "" (at 106.68 139.7 0) (effects (font (size 1 1)) (hide yes)))
